File: 2024-Semester-1/OIP/LB/led_control_system/led_control_system.kicad_sch (KiCad schematic)
At the start: 18 parts, among them Q1 BC547, Q2 BC547, Q3 BC547, Q4 BC547, Q5 BC547

Commit message: ОИП ЛБ 29.10.2024
Parts:
- C1: footprint (none) -> Capacitor_SMD:C_1210_3225Metric
- D1, D2, D3, D4: footprint (none) -> LED_THT:LED_D8.0mm
- MK1: footprint (none) -> Sensor_Audio:CUI_CMC-4013-SMT
- R1, R2, R3, R4, R5, R6, R7: footprint (none) -> Resistor_SMD:R_1210_3225Metric
Changed lines of the file:
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@@
 			)
 		)
-		(property "Footprint" ""
+		(property "Footprint" "Sensor_Audio:CUI_CMC-4013-SMT"
 			(at 66.04 105.41 90)
 			(effects
@@
 			)
 		)
-		(property "Footprint" ""
+		(property "Footprint" "LED_THT:LED_D8.0mm"
 			(at 139.7 63.5 0)
 			(effects
@@
 			)
 		)
-		(property "Footprint" ""
+		(property "Footprint" "Resistor_SMD:R_1210_3225Metric"
 			(at 101.092 63.5 90)
 			(effects
@@
 			)
 		)
-		(property "Footprint" ""
+		(property "Footprint" "LED_THT:LED_D8.0mm"
 			(at 177.8 63.5 0)
 			(effects
@@
 			)
 		)
-		(property "Footprint" ""
+		(property "Footprint" "Resistor_SMD:R_1210_3225Metric"
 			(at 176.022 107.95 90)
 			(effects
@@
 			)
 		)
-		(property "Footprint" ""
+		(property "Footprint" "Resistor_SMD:R_1210_3225Metric"
 			(at 137.922 107.95 90)
 			(effects
@@
 			)
 		)
-		(property "Footprint" ""
+		(property "Footprint" "LED_THT:LED_D8.0mm"
 			(at 120.65 63.5 0)
 			(effects
@@
 			)
 		)
-		(property "Footprint" ""
+		(property "Footprint" "Resistor_SMD:R_1210_3225Metric"
 			(at 82.042 63.5 90)
 			(effects
@@
 			)
 		)
-		(property "Footprint" ""
+		(property "Footprint" "Resistor_SMD:R_1210_3225Metric"
 			(at 118.872 107.95 90)
 			(effects
@@
 			)
 		)
-		(property "Footprint" ""
+		(property "Footprint" "Capacitor_SMD:C_1210_3225Metric"
 			(at 80.01 86.6648 0)
 			(effects
@@
 			)
 		)
-		(property "Footprint" ""
+		(property "Footprint" "LED_THT:LED_D8.0mm"
 			(at 158.75 63.5 0)
 			(effects
@@
 			)
 		)
-		(property "Footprint" ""
+		(property "Footprint" "Resistor_SMD:R_1210_3225Metric"
 			(at 156.972 107.95 90)
 			(effects
@@
 			)
 		)
-		(property "Footprint" ""
+		(property "Footprint" "Resistor_SMD:R_1210_3225Metric"
 			(at 64.262 63.5 90)
 			(effects
